File: Hardware/C5V1/C5V1/C5V1.sch (KiCad schematic (older format))
At the start: 0 parts

Commit message: Dodano schemat ISN
Changed lines of the file:
@@
 $Descr A4 11693 8268
 encoding utf-8
-Sheet 1 2
+Sheet 1 4
 Title ""
 Date ""
@@
 F1 "Procek1.sch" 50
 $EndSheet
+$Sheet
+S 4900 1250 1550 1600
+U 64512A12
+F0 "ISM330ISN" 50
+F1 "ISM330ISN.sch" 50
+$EndSheet
+$Sheet
+S 7300 1250 1650 1600
+U 6451B38A
+F0 "BME688" 50
+F1 "BME688.sch" 50
+$EndSheet
 $EndSCHEMATC
