File: Hardware/C5V1/C5V1/Procek1.sch (KiCad schematic (older format))
At the start: 1 part, among them IC1 STM32H725ZGT6

Commit message: Dodano początkowe zasilanie
Parts:
- added C? (x6): C, symbol Device:C
- added L?: L, symbol Device:L
- added R?: R, symbol Device:R
- renumbered IC1 to U?
Connections:
- net GND: now reaches U?.14 (VSSSMPS)
- net GND: now also U?.18 (VSS_3), U?.33 (VSS_4), U?.34 (VSSA), C?.1, C?.1, C?.1, C?.2, C?.2, C?.2
- net VLXSMPS: now reaches U?.15 (VLXSMPS)
- net VLXSMPS: now also L?.2
- net +3V3: now reaches U?.16 (VDDSMPS)
- net +3V3: now also U?.19 (VDD_3), U?.32 (VDD_4), U?.36 (VDDA), C?.1, C?.2, C?.2, C?.2, R?.1
- net VFBSMPS: now reaches U?.17 (VFBSMPS)
- net VFBSMPS: now also C?.1, C?.1, L?.1
- net VREF: now reaches U?.35 (VREF+)
- net VREF: now also R?.2
Other:
- note added: "SMPS"

Commit message: Dodano schemat ISN
Parts:
- C1, C2, C3, C4, C5, C6: renamed from C?; footprint (none) -> Capacitor_SMD:C_0402_1005Metric
- R1: renamed from R?; footprint (none) -> Resistor_SMD:R_0402_1005Metric
- gave numbers to parts that had none: 2
Changed lines of the file:
@@
 $Descr A1 33110 23386
 encoding utf-8
-Sheet 2 2
+Sheet 2 4
 Title ""
 Date ""
@@
 $EndDescr
 $Comp
-L STM32H725ZGT6:STM32H725ZGT6 U?
+L STM32H725ZGT6:STM32H725ZGT6 U1
 U 1 1 64450802
 P 11600 5450
-F 0 "U?" H 15744 3746 50  0000 L CNN
+F 0 "U1" H 15744 3746 50  0000 L CNN
 F 1 "STM32H725ZGT6" H 15744 3655 50  0000 L CNN
 F 2 "QFP50P2200X2200X160-144N" H 15550 6050 50  0001 L CNN
@@
 $EndComp
 $Comp
-L Device:L L?
+L Device:L L1
 U 1 1 64465B7B
 P 7700 2650
-F 0 "L?" V 7890 2650 50  0000 C CNN
+F 0 "L1" V 7890 2650 50  0000 C CNN
 F 1 "L" V 7799 2650 50  0000 C CNN
 F 2 "" H 7700 2650 50  0001 C CNN
@@
 SMPS
 $Comp
-L Device:C C?
+L Device:C C2
 U 1 1 64469018
 P 7400 2900
-F 0 "C?" H 7515 2946 50  0000 L CNN
+F 0 "C2" H 7515 2946 50  0000 L CNN
 F 1 "C" H 7515 2855 50  0000 L CNN
-F 2 "" H 7438 2750 50  0001 C CNN
+F 2 "Capacitor_SMD:C_0402_1005Metric" H 7438 2750 50  0001 C CNN
 F 3 "~" H 7400 2900 50  0001 C CNN
 	1    7400 2900
@@
 $EndComp
 $Comp
-L Device:C C?
+L Device:C C1
 U 1 1 64469E26
 P 7100 2900
-F 0 "C?" H 7215 2946 50  0000 L CNN
+F 0 "C1" H 7215 2946 50  0000 L CNN
 F 1 "C" H 7215 2855 50  0000 L CNN
-F 2 "" H 7138 2750 50  0001 C CNN
+F 2 "Capacitor_SMD:C_0402_1005Metric" H 7138 2750 50  0001 C CNN
 F 3 "~" H 7100 2900 50  0001 C CNN
 	1    7100 2900
@@
 	7250 3050 7100 3050
 $Comp
-L power:GND #PWR?
+L power:GND #PWR0101
 U 1 1 6446A970
 P 7250 3200
-F 0 "#PWR?" H 7250 2950 50  0001 C CNN
+F 0 "#PWR0101" H 7250 2950 50  0001 C CNN
 F 1 "GND" H 7255 3027 50  0000 C CNN
 F 2 "" H 7250 3200 50  0001 C CNN
@@
 	10800 6950 10800 6850
 $Comp
-L power:+3V3 #PWR?
+L power:+3V3 #PWR0102
 U 1 1 6446C5F3
 P 10800 6650
-F 0 "#PWR?" H 10800 6500 50  0001 C CNN
+F 0 "#PWR0102" H 10800 6500 50  0001 C CNN
 F 1 "+3V3" H 10815 6823 50  0000 C CNN
 F 2 "" H 10800 6650 50  0001 C CNN
@@
 $EndComp
 $Comp
-L Device:C C?
+L Device:C C5
 U 1 1 6446DA73
 P 10800 7200
-F 0 "C?" H 10800 7200 50  0000 L CNN
+F 0 "C5" H 10800 7200 50  0000 L CNN
 F 1 "C" H 10700 7200 50  0000 L CNN
-F 2 "" H 10838 7050 50  0001 C CNN
+F 2 "Capacitor_SMD:C_0402_1005Metric" H 10838 7050 50  0001 C CNN
 F 3 "~" H 10800 7200 50  0001 C CNN
 	1    10800 7200
@@
 Connection ~ 10800 7050
 $Comp
-L power:GND #PWR?
+L power:GND #PWR0103
 U 1 1 6446F587
 P 10550 7100
-F 0 "#PWR?" H 10550 6850 50  0001 C CNN
+F 0 "#PWR0103" H 10550 6850 50  0001 C CNN
 F 1 "GND" H 10555 6927 50  0000 C CNN
 F 2 "" H 10550 7100 50  0001 C CNN
@@
 	11050 6750 11050 6800
 $Comp
-L power:GND #PWR?
+L power:GND #PWR0104
 U 1 1 64470EA1
 P 11050 6800
-F 0 "#PWR?" H 11050 6550 50  0001 C CNN
+F 0 "#PWR0104" H 11050 6550 50  0001 C CNN
 F 1 "GND" H 11050 6900 50  0000 C CNN
 F 2 "" H 11050 6800 50  0001 C CNN
@@
 $EndComp
 $Comp
-L Device:C C?
+L Device:C C6
 U 1 1 6447150B
 P 11050 8600
-F 0 "C?" H 11165 8646 50  0000 L CNN
+F 0 "C6" H 11165 8646 50  0000 L CNN
 F 1 "C" H 11165 8555 50  0000 L CNN
-F 2 "" H 11088 8450 50  0001 C CNN
+F 2 "Capacitor_SMD:C_0402_1005Metric" H 11088 8450 50  0001 C CNN
 F 3 "~" H 11050 8600 50  0001 C CNN
 	1    11050 8600
@@
 	11250 8750 11050 8750
 $Comp
-L power:GND #PWR?
+L power:GND #PWR0105
 U 1 1 64472CF9
 P 11050 8750
-F 0 "#PWR?" H 11050 8500 50  0001 C CNN
+F 0 "#PWR0105" H 11050 8500 50  0001 C CNN
 F 1 "GND" H 11055 8577 50  0000 C CNN
 F 2 "" H 11050 8750 50  0001 C CNN
@@
 Connection ~ 11050 8750
 $Comp
-L power:+3V3 #PWR?
+L power:+3V3 #PWR0106
 U 1 1 644733E5
 P 11050 8450
-F 0 "#PWR?" H 11050 8300 50  0001 C CNN
+F 0 "#PWR0106" H 11050 8300 50  0001 C CNN
 F 1 "+3V3" H 11065 8623 50  0000 C CNN
 F 2 "" H 11050 8450 50  0001 C CNN
@@
 	11600 8950 11600 9200
 $Comp
-L Device:C C?
+L Device:C C4
 U 1 1 64475B86
 P 10350 9100
-F 0 "C?" H 10465 9146 50  0000 L CNN
+F 0 "C4" H 10465 9146 50  0000 L CNN
 F 1 "C" H 10465 9055 50  0000 L CNN
-F 2 "" H 10388 8950 50  0001 C CNN
+F 2 "Capacitor_SMD:C_0402_1005Metric" H 10388 8950 50  0001 C CNN
 F 3 "~" H 10350 9100 50  0001 C CNN
 	1    10350 9100
@@
 	10550 9000 11350 9000
 $Comp
-L Device:C C?
+L Device:C C3
 U 1 1 64476D9C
 P 10050 9100
-F 0 "C?" H 10165 9146 50  0000 L CNN
+F 0 "C3" H 10165 9146 50  0000 L CNN
 F 1 "C" H 10165 9055 50  0000 L CNN
-F 2 "" H 10088 8950 50  0001 C CNN
+F 2 "Capacitor_SMD:C_0402_1005Metric" H 10088 8950 50  0001 C CNN
 F 3 "~" H 10050 9100 50  0001 C CNN
 	1    10050 9100
@@
 Connection ~ 10350 9300
 $Comp
-L power:+3V3 #PWR?
+L power:+3V3 #PWR0107
 U 1 1 6447B7BF
 P 10050 9250
-F 0 "#PWR?" H 10050 9100 50  0001 C CNN
+F 0 "#PWR0107" H 10050 9100 50  0001 C CNN
 F 1 "+3V3" H 10065 9423 50  0000 C CNN
 F 2 "" H 10050 9250 50  0001 C CNN
@@
 Connection ~ 10050 9250
 $Comp
-L power:GND #PWR?
+L power:GND #PWR0108
 U 1 1 6447E958
 P 10050 8900
-F 0 "#PWR?" H 10050 8650 50  0001 C CNN
+F 0 "#PWR0108" H 10050 8650 50  0001 C CNN
 F 1 "GND" H 10055 8727 50  0000 C CNN
 F 2 "" H 10050 8900 50  0001 C CNN
@@
 	11450 8850 11450 9550
 $Comp
-L Device:R R?
+L Device:R R1
 U 1 1 6448256F
 P 10800 9350
-F 0 "R?" H 10870 9396 50  0000 L CNN
+F 0 "R1" H 10870 9396 50  0000 L CNN
 F 1 "R" H 10870 9305 50  0000 L CNN
-F 2 "" V 10730 9350 50  0001 C CNN
+F 2 "Resistor_SMD:R_0402_1005Metric" V 10730 9350 50  0001 C CNN
 F 3 "~" H 10800 9350 50  0001 C CNN
 	1    10800 9350
