File: Hardware/C5V1/C5V1/_autosave-C5V1.kicad_pcb (KiCad board)
At the start: 2 copper layers, 0 parts

Commit message: Dodano schemat ISN
Parts:
- added C1: C, Capacitor_SMD:C_0402_1005Metric, F.Cu at (150.8, 63.8)
- added C10: C, Capacitor_SMD:C_0402_1005Metric, F.Cu at (157.1, 79.2)
- added C11: C, Capacitor_SMD:C_0402_1005Metric, F.Cu at (160.0, 77.2)
- added C12: C, Capacitor_SMD:C_0402_1005Metric, F.Cu at (160.0, 79.2)
- added C13: C, Capacitor_SMD:C_0402_1005Metric, F.Cu at (162.8, 77.2)
- added C2: C, Capacitor_SMD:C_0402_1005Metric, F.Cu at (150.8, 65.8)
- added C3: C, Capacitor_SMD:C_0402_1005Metric, F.Cu at (153.7, 63.8)
- added C4: C, Capacitor_SMD:C_0402_1005Metric, F.Cu at (150.8, 67.8)
- added C5: C, Capacitor_SMD:C_0402_1005Metric, F.Cu at (153.7, 65.8)
- added C6: C, Capacitor_SMD:C_0402_1005Metric, F.Cu at (156.5, 63.8)
- added C7: 100n/10V/X5R, Capacitor_SMD:C_0402_1005Metric, F.Cu at (178.8, 63.8)
- added C8: 100n/10V/X5R, Capacitor_SMD:C_0402_1005Metric, F.Cu at (178.8, 65.8)
- added C9: C, Capacitor_SMD:C_0402_1005Metric, F.Cu at (157.1, 77.2)
- added R1: R, Capacitor_SMD:C_0402_1005Metric, F.Cu at (150.8, 69.8)
- added U1: STM32H725ZGT6, C5V1:QFP50P2200X2200X160-144N, F.Cu at (135.8, 70.9)
- added U2: ISM330ISN, Package_LGA:LGA-14_3x2.5mm_P0.5mm_LayoutBorder3x4y, F.Cu at (158.4, 70.4)
