File: Hardware/C5V1/C5V1/_autosave-Procek1.sch (KiCad schematic (older format))
At the start: 9 parts, among them U1 STM32H725ZGT6

Commit message: Dodano schemat ISN
Parts:
- added C10, C11, C12, C13, C9: C, Capacitor_SMD:C_0402_1005Metric, symbol Device:C
- R1: footprint Capacitor_SMD:C_0402_1005Metric -> Resistor_SMD:R_0402_1005Metric
Connections:
- net +3V3: now also U1.119 (VDD_11), U1.129 (VDD_12), U1.42 (VDD_5), U1.56 (VDD_6), U1.80 (VSS_8), C10.1, C11.1, C12.1, C13.1, C9.1
- net GND: now also U1.118 (VSS_11), U1.128 (VSS_12), U1.41 (VSS_5), U1.55 (VSS_6), U1.79 (VDD_8), C10.2, C11.2, C12.2, C13.2, C9.2
