File: Hardware/C5W1B1V1.0/Screen.sch (KiCad schematic (older format))
At the start: 0 parts

Commit message: Rozlana masa
Parts:
- added C60: 100n/16V/X5R, Capacitor_SMD:C_0402_1005Metric, symbol Device:C
- added J6: Conn_01x08_Male, Connector_PinHeader_2.54mm:PinHeader_1x08_P2.54mm_Vertical, symbol Connector:Conn_01x08_Male
Connections:
- new net +3V3: C60.2, J6.8 (Pin_8)
- new net GND: C60.1, J6.7 (Pin_7)
- new net SSD1331_CS: J6.3 (Pin_3)
- new net SSD1331_DC: J6.2 (Pin_2)
- new net SSD1331_MOSI: J6.5 (Pin_5)
- new net SSD1331_RES: J6.1 (Pin_1)
- new net SSD1331_SCK: J6.4 (Pin_4)
- no-connect marks 0 -> 1
Changed lines of the file:
@@
 $Descr A4 11693 8268
 encoding utf-8
-Sheet 1 8
+Sheet 7 8
 Title ""
 Date ""
@@
 Comment4 ""
 $EndDescr
+$Comp
+L Connector:Conn_01x08_Male J6
+U 1 1 66906C5E
+P 1950 1600
+F 0 "J6" H 2058 2081 50  0000 C CNN
+F 1 "Conn_01x08_Male" H 2058 1990 50  0000 C CNN
+F 2 "Connector_PinHeader_2.54mm:PinHeader_1x08_P2.54mm_Vertical" H 1950 1600 50  0001 C CNN
+F 3 "~" H 1950 1600 50  0001 C CNN
+	1    1950 1600
+	-1   0    0    1
+$EndComp
+Text GLabel 1750 1600 0    50   Input ~ 0
+SSD1331_SCK
+Text GLabel 1750 1800 0    50   Input ~ 0
+SSD1331_DC
+Text GLabel 1750 1900 0    50   Input ~ 0
+SSD1331_RES
+Text GLabel 1750 1500 0    50   Input ~ 0
+SSD1331_MOSI
+Text GLabel 1750 1700 0    50   Input ~ 0
+SSD1331_CS
+NoConn ~ 1750 1400
+Wire Wire Line
+	1750 1300 850  1300
+Wire Wire Line
+	850  1300 850  1400
+$Comp
+L power:GND #PWR0256
+U 1 1 66AFB2B0
+P 850 1650
+F 0 "#PWR0256" H 850 1400 50  0001 C CNN
+F 1 "GND" H 855 1477 50  0000 C CNN
+F 2 "" H 850 1650 50  0001 C CNN
+F 3 "" H 850 1650 50  0001 C CNN
+	1    850  1650
+	1    0    0    -1
+$EndComp
+Wire Wire Line
+	1750 1200 850  1200
+Wire Wire Line
+	850  1200 850  1100
+$Comp
+L power:+3V3 #PWR0257
+U 1 1 66AFBAFC
+P 850 1000
+F 0 "#PWR0257" H 850 850 50  0001 C CNN
+F 1 "+3V3" H 865 1173 50  0000 C CNN
+F 2 "" H 850 1000 50  0001 C CNN
+F 3 "" H 850 1000 50  0001 C CNN
+	1    850  1000
+	1    0    0    -1
+$EndComp
+$Comp
+L Device:C C?
+U 1 1 66AFE7CB
+P 700 1250
+AR Path="/665B4F23/66AFE7CB" Ref="C?"  Part="1"
+AR Path="/66C17F09/66AFE7CB" Ref="C60"  Part="1"
+F 0 "C60" H 800 1350 50  0000 L CNN
+F 1 "100n/16V/X5R" H 850 1250 50  0000 L CNN
+F 2 "Capacitor_SMD:C_0402_1005Metric" H 738 1100 50  0001 C CNN
+F 3 "~" H 700 1250 50  0001 C CNN
+	1    700  1250
+	-1   0    0    1
+$EndComp
+Wire Wire Line
+	700  1100 850  1100
+Connection ~ 850  1100
+Wire Wire Line
+	850  1100 850  1000
+Wire Wire Line
+	850  1400 700  1400
+Connection ~ 850  1400
+Wire Wire Line
+	850  1400 850  1650
 $EndSCHEMATC
