File: Hardware/C5W1B1V1.0/ESP.sch (KiCad schematic (older format))
At the start: 17 parts, among them IC1 ESP32-C3-WROOM-02-N4, SW3 SW_Push_Dual, SW4 SW_Push_Dual, Y3 830106545501

Commit message: Rozlana masa
Parts:
- renumbered IC1 to U12
Connections:
- net STM_ESP_PIN2: no longer names the net of U12.15 (IO3)
- no-connect marks 0 -> 1
Changed lines of the file:
@@
 $EndDescr
 $Comp
-L ESP32-C3-WROOM-02-N4:ESP32-C3-WROOM-02-N4 IC1
+L ESP32-C3-WROOM-02-N4:ESP32-C3-WROOM-02-N4 U12
 U 1 1 676EB2F3
 P 9100 3800
-F 0 "IC1" H 9750 4065 50  0000 C CNN
+F 0 "U12" H 9750 4065 50  0000 C CNN
 F 1 "ESP32-C3-WROOM-02-N4" H 9750 3974 50  0000 C CNN
 F 2 "ESP32C3WROOM02N4" H 10250 3900 50  0001 L CNN
@@
 Text GLabel 9100 4300 0    50   BiDi ~ 0
 STM_ESP_PIN1
-Text GLabel 10400 3800 2    50   BiDi ~ 0
-STM_ESP_PIN2
 Wire Wire Line
 	6900 3900 6900 2750
@@
 Wire Wire Line
 	11400 4300 12500 4300
+NoConn ~ 10400 3800
 $EndSCHEMATC

Commit message: End PCB
Connections:
- net STM_ESP_PIN2: now reaches U12.15 (IO3)
- no-connect marks 1 -> 0
Changed lines of the file:
@@
 Wire Wire Line
 	11400 4300 12500 4300
-NoConn ~ 10400 3800
+Text GLabel 10400 3650 1    50   BiDi ~ 0
+STM_ESP_PIN2
+Wire Wire Line
+	10400 3800 10400 3650
 $EndSCHEMATC
