File: Hardware/C5W1B1V1.0/Kicad/C5W1B1V1.0.kicad_pcb (KiCad board)
At the start: 4 copper layers, 100 x 100 mm, 149 parts, among them J1 Conn_02x20_Counter_Clockwise, J2 Conn_02x20_Counter_Clockwise, J3 Conn_01x13_Male, J4 Conn_01x04, J5 USB4105GFA120, J6 Conn_01x08_Male, J7 Conn_01x02_Male, J8 Conn_01x02_Male, SW1 SW_Push_Dual, SW2 SW_Push_Dual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

Commit message: Dodano mikrofony i więcej WS2812B
Parts:
- added C75: 100n/16V/X5R, Capacitor_SMD:C_0402_1005Metric, F.Cu at (119.6, 104.6)
- added C76: 100n/16V/X5R, Capacitor_SMD:C_0402_1005Metric, F.Cu at (114.0, 104.6)
- added C77: 100n/16V/X5R, Capacitor_SMD:C_0402_1005Metric, F.Cu at (72.1, 121.7)
- added C78: 1u/16V/X5R, Capacitor_SMD:C_0402_1005Metric, F.Cu at (72.1, 122.7)
- added C79: 100n/16V/X5R, Capacitor_SMD:C_0402_1005Metric, F.Cu at (77.5, 121.7)
- added C80: 1u/16V/X5R, Capacitor_SMD:C_0402_1005Metric, F.Cu at (77.5, 122.7)
- added D10: WS2812B, LED_SMD:LED_WS2812B_PLCC4_5.0x5.0mm_P3.2mm, F.Cu at (120.7, 100.6)
- added D11: WS2812B, LED_SMD:LED_WS2812B_PLCC4_5.0x5.0mm_P3.2mm, F.Cu at (115.1, 100.6)
- added MK1: MP34DT05TR-A, Footprints:MP34DT05TRA, F.Cu at (71.7, 118.2)
- added MK2: MP34DT05TR-A, Footprints:MP34DT05TRA, F.Cu at (76.8, 118.2)
- added R34: 100k/5%/0.063W, Resistor_SMD:R_0402_1005Metric, F.Cu at (72.3, 114.6)
- added R35: 100k/5%/0.063W, Resistor_SMD:R_0402_1005Metric, F.Cu at (77.2, 114.5)
- moved C73 48.6 mm to (111.8, 93.2)
- moved C72 47.1 mm to (111.8, 90.8)
- moved C70 47.0 mm to (111.7, 88.5)
- moved C71 45.6 mm to (111.8, 95.6)
- moved R18 7.89 mm to (122.2, 127.2)
- moved R26 5.53 mm to (124.2, 96.6)
- moved D6 4.10 mm to (126.3, 100.6)
- moved C59 4.10 mm to (125.3, 104.5)
Connections:
- J2 pad 17: PE7 -> GND
- J2 pad 19: PE9 -> +3V3
- J2 pad 38: 5V_USB -> +5V
- U1 pad 67: PE7 -> DFSDM_DATA
- U1 pad 69: PE9 -> DFSDM_CLK
Routing:
- net +5V: track 191.9 -> 243.4 mm, vias 6 -> 2
- net 5V_USB: track 68.6 -> 19.7 mm, vias 2 -> 0
- net PE9: track 41.2 -> 0.00 mm, vias 2 -> 0
- net PE7: track 36.5 -> 0.00 mm, vias 2 -> 0
- net DFSDM_CLK: track 0.00 -> 34.2 mm, vias 0 -> 4
- net DFSDM_DATA: track 0.00 -> 22.4 mm, vias 0 -> 4
- net Net-(D10-Pad2): track 0.00 -> 18.8 mm
- net BUTTON1: track 59.9 -> 71.8 mm
- net Net-(D10-Pad4): track 0.00 -> 10.8 mm
- net +3V3: track 128.1 -> 137.9 mm, vias 70 -> 72
- net Net-(MK2-Pad2): track 0.00 -> 9.06 mm, vias 0 -> 2
- net Net-(MK1-Pad2): track 0.00 -> 8.49 mm
- net LED2: track 45.5 -> 51.1 mm
- net WS2812: track 42.7 -> 37.8 mm
- net BUTTON2: track 69.1 -> 73.1 mm
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Other:
- board text added: "."
- board text removed: "PE7"
- board text removed: "PE9"
