File: Hardware/C5W1B1V1.0/Kicad/C5W1B1V1.0.sch (KiCad schematic (older format))
At the start: 0 parts

Commit message: Dodano mikrofony i więcej WS2812B
Changed lines of the file:
@@
 $Descr A4 11693 8268
 encoding utf-8
-Sheet 1 8
+Sheet 1 9
 Title ""
 Date ""
@@
 F1 "ESP.sch" 50
 $EndSheet
+$Sheet
+S 4450 2800 1650 1500
+U 6737B7AB
+F0 "Audio" 50
+F1 "Audio.sch" 50
+$EndSheet
 $EndSCHEMATC
