File: Hardware/C5W1B1V1.0/Kicad/ESP.sch (KiCad schematic (older format))
At the start: 22 parts, among them SW3 SW_Push_Dual, SW4 SW_Push_Dual, U12 ESP32-C3-WROOM-02-N4, Y3 830106545501

Commit message: Drobne poprawki
Parts:
- C38, C39: value 6p/16V/COG -> 8p/16V/COG
Changed lines of the file:
@@
 AR Path="/676EAB19/66BBDDAF" Ref="C39"  Part="1"
 F 0 "C39" H 13115 4346 50  0000 L CNN
-F 1 "6p/16V/COG" H 13115 4255 50  0000 L CNN
+F 1 "8p/16V/COG" H 13115 4255 50  0000 L CNN
 F 2 "Capacitor_SMD:C_0402_1005Metric" H 13038 4150 50  0001 C CNN
 F 3 "~" H 13000 4300 50  0001 C CNN
@@
 AR Path="/676EAB19/66BBDDB5" Ref="C38"  Part="1"
 F 0 "C38" H 13115 4046 50  0000 L CNN
-F 1 "6p/16V/COG" H 13115 3955 50  0000 L CNN
+F 1 "8p/16V/COG" H 13115 3955 50  0000 L CNN
 F 2 "Capacitor_SMD:C_0402_1005Metric" H 13038 3850 50  0001 C CNN
 F 3 "~" H 13000 4000 50  0001 C CNN
