File: Hardware/C5W1B1V1.0/Kicad/uC.sch (KiCad schematic (older format))
At the start: 61 parts, among them J3 Conn_01x13_Male, J7 Conn_01x02_Male, SW1 SW_Push_Dual, SW2 SW_Push_Dual, SW5 SW_Push_Dual, SW6 SW_Push_Dual, U1 STM32H735IGT6, Y1 ECS-250-8-36CKM-TR3, Y2 830106545501

Commit message: Dodano mikrofony i więcej WS2812B
Parts:
- added C75, C76: 100n/16V/X5R, Capacitor_SMD:C_0402_1005Metric, symbol Device:C
- added D10, D11: WS2812B, LED_SMD:LED_WS2812B_PLCC4_5.0x5.0mm_P3.2mm, symbol LED:WS2812B
Connections:
- net +5V: now also C75.1, C76.1, D10.1 (VDD), D11.1 (VDD)
- net GND: now also C75.2, C76.2, D10.3 (VSS), D11.3 (VSS)
- net at D6.2 (DOUT): now also D10.4 (DIN)
- net PE7 renamed DFSDM_DATA
- net PE9 renamed DFSDM_CLK
- new net: D10.2 (DOUT), D11.4 (DIN)
Other:
- moved on the sheet: C13, D4, D5, R27, R28

Commit message: Drobne poprawki
Parts:
- C26: value 6p/16V/COG -> 8pp/16V/COG
- C27: value 6p/16V/COG -> 8p/16V/COG
Changed lines of the file:
@@
 P 5650 6800
 F 0 "C26" H 5765 6846 50  0000 L CNN
-F 1 "6p/16V/COG" H 5765 6755 50  0000 L CNN
+F 1 "8pp/16V/COG" H 5765 6755 50  0000 L CNN
 F 2 "Capacitor_SMD:C_0402_1005Metric" H 5688 6650 50  0001 C CNN
 F 3 "~" H 5650 6800 50  0001 C CNN
@@
 P 5650 7100
 F 0 "C27" H 5765 7146 50  0000 L CNN
-F 1 "6p/16V/COG" H 5765 7055 50  0000 L CNN
+F 1 "8p/16V/COG" H 5765 7055 50  0000 L CNN
 F 2 "Capacitor_SMD:C_0402_1005Metric" H 5688 6950 50  0001 C CNN
 F 3 "~" H 5650 7100 50  0001 C CNN
